Commit message: Fix ros2_control xacro files.

File: orbita3d_description/ros2_control/orbita3d.ros2_control.xacro (robot description, xacro)
@@ -22,11 +22,11 @@
                 </xacro:if>
             </hardware>
-            <xacro:orbita3d_actuator_control name="{name}"/>
+            <xacro:orbita3d_actuator_control name="${name}"/>
             <xacro:orbita3d_axis_control name="${name}_roll"/>
             <xacro:orbita3d_axis_control name="${name}_pitch"/>
             <xacro:orbita3d_axis_control name="${name}_yaw"/>
-            <xacro:orbita3d_raw_motor_control name="${name}_motor_1"/>
-            <xacro:orbita3d_raw_motor_control name="${name}_motor_2"/>
-            <xacro:orbita3d_raw_motor_control name="${name}_motor_3"/>
+            <xacro:orbita3d_raw_motor_control name="${name}_raw_motor_1"/>
+            <xacro:orbita3d_raw_motor_control name="${name}_raw_motor_2"/>
+            <xacro:orbita3d_raw_motor_control name="${name}_raw_motor_3"/>
         </ros2_control>
     </xacro:macro>

File: orbita3d_description/ros2_control/orbita3d_actuator_control.ros2_control.xacro (robot description, xacro)
@@ -2,9 +2,10 @@
 <robot xmlns:xacro="http://www.ros.org/wiki/xacro">
   <xacro:macro name="orbita3d_actuator_control" params="name">
+    <gpio name="${name}">
       <state_interface name="torque">
         <param name="initial_value">0.0</param>
       </state_interface>
       <command_interface name="torque"/>
-    </joint>
+    </gpio>
   </xacro:macro>
 </robot>

File: orbita3d_description/ros2_control/orbita3d_raw_motor_control.ros2_control.xacro (robot description, xacro)
@@ -1,6 +1,6 @@
 <?xml version="1.0" ?>
 <robot xmlns:xacro="http://www.ros.org/wiki/xacro">
-  <xacro:macro name="orbita3d_actuator_control" params="name">
-      <gpio>
+  <xacro:macro name="orbita3d_raw_motor_control" params="name">
+      <gpio name="${name}">
         <state_interface name="speed_limit"/>
         <command_interface name="speed_limit"/>
@@ -14,5 +14,4 @@
         <command_interface name="d_gain"/>
       </gpio>
-    </joint>
   </xacro:macro>
 </robot>

Commit message: add errors

File: orbita3d_description/ros2_control/orbita3d.ros2_control.xacro (robot description, xacro)
@@ -4,34 +4,35 @@
   <xacro:include filename="$(find orbita3d_description)/ros2_control/orbita3d_axis_control.ros2_control.xacro"/>
   <xacro:include filename="$(find orbita3d_description)/ros2_control/orbita3d_raw_motor_control.ros2_control.xacro"/>
-    <xacro:macro name="orbita3d_control" params="name config_file">
-        <ros2_control name="${name}" type="system">
-            <hardware>
-                <xacro:unless value="$(arg use_fake_hardware)">
-                  <plugin>orbita3d_system_hwi/Orbita3dSystem</plugin>
-                    <param name="config_file">${config_file}</param>
-                </xacro:unless>
-                <xacro:if value="$(arg use_fake_hardware)">
-                    <!-- Use gazebo as hardware simulation. -->
-                    <xacro:if value="$(arg use_gazebo)">
-                        <plugin>gazebo_ros2_control/GazeboSystem</plugin>
-                    </xacro:if>
-                    <!-- Use fake components. -->
-                    <xacro:unless value="$(arg use_gazebo)">
-		      <!-- Standard ROS fake system -->
-                        <!-- <plugin>fake_components/GenericSystem</plugin> -->
-			<!-- Pollen controller fake system -->
-			<plugin>orbita3d_system_hwi/Orbita3dSystem</plugin>
-			<param name="config_file">${config_file}</param>
-                    </xacro:unless>
-                </xacro:if>
-            </hardware>
-            <xacro:orbita3d_actuator_control name="${name}"/>
-            <xacro:orbita3d_axis_control name="${name}_roll"/>
-            <xacro:orbita3d_axis_control name="${name}_pitch"/>
-            <xacro:orbita3d_axis_control name="${name}_yaw"/>
-            <xacro:orbita3d_raw_motor_control name="${name}_raw_motor_1"/>
-            <xacro:orbita3d_raw_motor_control name="${name}_raw_motor_2"/>
-            <xacro:orbita3d_raw_motor_control name="${name}_raw_motor_3"/>
-        </ros2_control>
-    </xacro:macro>
+  <xacro:macro name="orbita3d_control" params="name config_file">
+    <ros2_control name="${name}" type="system">
+      <hardware>
+        <!-- Use real hardware. -->
+        <xacro:unless value="$(arg use_fake_hardware)">
+          <plugin>orbita3d_system_hwi/Orbita3dSystem</plugin>
+          <param name="config_file">${config_file}</param>
+        </xacro:unless>
+        <xacro:if value="$(arg use_fake_hardware)">
+          <!-- Use gazebo as hardware simulation. -->
+          <xacro:if value="$(arg use_gazebo)">
+            <plugin>gazebo_ros2_control/GazeboSystem</plugin>
+          </xacro:if>
+          <!-- Use fake components. -->
+          <xacro:unless value="$(arg use_gazebo)">
+	    <!-- Standard ROS fake system -->
+            <!-- <plugin>fake_components/GenericSystem</plugin> -->
+	    <!-- Pollen controller fake system -->
+	    <plugin>orbita3d_system_hwi/Orbita3dSystem</plugin>
+	    <param name="config_file">${config_file}</param>
+          </xacro:unless>
+        </xacro:if>
+      </hardware>
+      <xacro:orbita3d_actuator_control name="${name}"/>
+      <xacro:orbita3d_axis_control name="${name}_roll"/>
+      <xacro:orbita3d_axis_control name="${name}_pitch"/>
+      <xacro:orbita3d_axis_control name="${name}_yaw"/>
+      <xacro:orbita3d_raw_motor_control name="${name}_raw_motor_1"/>
+      <xacro:orbita3d_raw_motor_control name="${name}_raw_motor_2"/>
+      <xacro:orbita3d_raw_motor_control name="${name}_raw_motor_3"/>
+    </ros2_control>
+  </xacro:macro>
 </robot>

File: orbita3d_description/ros2_control/orbita3d_actuator_control.ros2_control.xacro (robot description, xacro)
@@ -6,4 +6,5 @@
         <param name="initial_value">0.0</param>
       </state_interface>
+      <state_interface name="errors" />
       <command_interface name="torque"/>
     </gpio>
