Commit message: add urdf and launch

File: orbita3d_description/urdf/orbita3d.urdf.xacro (robot description, xacro)
@@ -3,7 +3,5 @@
   <xacro:include filename="$(find pollen_generic_description)/urdf/inertial_primitives.urdf.xacro"/>
   <xacro:include filename="$(find orbita3d_description)/ros2_control/orbita3d.ros2_control.xacro"/>
-  <xacro:macro name="orbita3d" params="name parent length radius mass xyz rpy damping friction configfile">
-    <!-- 54°?? -->
-  <xacro:property name="orbita3d_alpha" value="0.9424777960769379"/>
+  <xacro:macro name="orbita3d" params="name parent length radius mass xyz rpy damping friction config_file">
     <material name="orbita3d_yellow">
         <color rgba="0.8 0.8 0.0 1"/>

Commit message: urdf stuff

File: orbita3d_description/urdf/orbita3d.urdf.xacro (robot description, xacro)
@@ -4,8 +4,8 @@
   <xacro:include filename="$(find orbita3d_description)/ros2_control/orbita3d.ros2_control.xacro"/>
   <xacro:macro name="orbita3d" params="name parent length radius mass xyz rpy damping friction config_file">
-    <material name="orbita3d_yellow">
+    <material name="${name}_orbita3d_yellow">
         <color rgba="0.8 0.8 0.0 1"/>
     </material>
-    <material name="orbita3d_grey">
+    <material name="${name}_orbita3d_grey">
         <color rgba="0.8 0.8 0.8 1"/>
     </material>
@@ -33,5 +33,5 @@
           <cylinder length="${length}" radius="${radius}"/>
       	</geometry>
-      	<material name="orbita3d_yellow"/>
+      	<material name="${name}_orbita3d_yellow"/>
       </visual>
       <collision>
@@ -50,5 +50,5 @@
           <sphere radius="${radius*1.2}"/>
       	</geometry>
-      	<material name="orbita3d_grey"/>
+      	<material name="${name}_orbita3d_grey"/>
       </visual>
       <collision>

Commit message: small change in urdf for colo

File: orbita3d_description/urdf/orbita3d.urdf.xacro (robot description, xacro)
@@ -2,12 +2,13 @@
 <robot xmlns:xacro="http://www.ros.org/wiki/xacro">
   <xacro:include filename="$(find pollen_generic_description)/urdf/inertial_primitives.urdf.xacro"/>
+  <xacro:include filename="$(find pollen_generic_description)/urdf/materials.urdf.xacro"/>
   <xacro:include filename="$(find orbita3d_description)/ros2_control/orbita3d.ros2_control.xacro"/>
   <xacro:macro name="orbita3d" params="name parent length radius mass xyz rpy damping friction config_file">
-    <material name="orbita3d_yellow">
-        <color rgba="0.8 0.8 0.0 1"/>
-    </material>
-    <material name="orbita3d_grey">
-        <color rgba="0.8 0.8 0.8 1"/>
-    </material>
+    <!-- <material name="orbita3d_yellow"> -->
+    <!--     <color rgba="0.8 0.8 0.0 1"/> -->
+    <!-- </material> -->
+    <!-- <material name="orbita3d_grey"> -->
+    <!--     <color rgba="0.8 0.8 0.8 1"/> -->
+    <!-- </material> -->
     <!--
       Orbita3d
@@ -33,5 +34,6 @@
           <cylinder length="${length}" radius="${radius}"/>
       	</geometry>
-      	<material name="orbita3d_yellow"/>
+      	<!-- <material name="orbita3d_yellow"/> -->
+	<xacro:orbita3d_yellow/>
       </visual>
       <collision>
@@ -50,5 +52,6 @@
           <sphere radius="${radius*1.2}"/>
       	</geometry>
-      	<material name="orbita3d_grey"/>
+      	<!-- <material name="orbita3d_grey"/> -->
+	<xacro:orbita3d_grey/>
       </visual>
       <collision>

Commit message: Clean up

File: orbita3d_description/urdf/orbita3d.urdf.xacro (robot description, xacro)
@@ -5,10 +5,4 @@
   <xacro:include filename="$(find orbita3d_description)/ros2_control/orbita3d.ros2_control.xacro"/>
   <xacro:macro name="orbita3d" params="name parent length radius mass xyz rpy damping friction config_file">
-    <!-- <material name="orbita3d_yellow"> -->
-    <!--     <color rgba="0.8 0.8 0.0 1"/> -->
-    <!-- </material> -->
-    <!-- <material name="orbita3d_grey"> -->
-    <!--     <color rgba="0.8 0.8 0.8 1"/> -->
-    <!-- </material> -->
     <!--
       Orbita3d
@@ -34,6 +28,5 @@
           <cylinder length="${length}" radius="${radius}"/>
       	</geometry>
-      	<!-- <material name="orbita3d_yellow"/> -->
-	<xacro:orbita3d_yellow/>
+      	<xacro:orbita3d_yellow/>
       </visual>
       <collision>
@@ -52,6 +45,5 @@
           <sphere radius="${radius*1.2}"/>
       	</geometry>
-      	<!-- <material name="orbita3d_grey"/> -->
-	<xacro:orbita3d_grey/>
+      	<xacro:orbita3d_grey/>
       </visual>
       <collision>

Commit message: update for neck

File: orbita3d_description/urdf/orbita3d.urdf.xacro (robot description, xacro)
@@ -23,35 +23,35 @@
     </link>
     <link name="${name}_link">
-      <visual>
-      	<origin xyz="0 0 ${length/2}" rpy="0 0 0"/>
-      	<geometry>
-          <cylinder length="${length}" radius="${radius}"/>
-      	</geometry>
-      	<xacro:orbita3d_yellow/>
-      </visual>
-      <collision>
-      	<origin xyz="0 0 ${length/2}" rpy="0 0 0"/>
-      	<geometry>
-          <cylinder length="${length}" radius="${radius}"/>
-      	</geometry>
-      </collision>
-      <xacro:inertial_cuboid mass="${mass*0.48}" xyz="0 0 ${-length/2}"  rpy="0 0 0" x_length="${radius*2}" y_length="${radius*2}" z_length="${length}">
+      <!-- <visual> -->
+      <!-- 	<origin xyz="0 0 0" rpy="0 0 0"/> -->
+      <!-- 	<geometry> -->
+      <!--     <cylinder length="${length}" radius="${radius}"/> -->
+      <!-- 	</geometry> -->
+      <!-- 	<xacro:orbita3d_grey/> -->
+      <!-- </visual> -->
+      <!-- <collision> -->
+      <!-- 	<origin xyz="0 0 ${length/2}" rpy="0 0 0"/> -->
+      <!-- 	<geometry> -->
+      <!--     <cylinder length="${length}" radius="${radius}"/> -->
+      <!-- 	</geometry> -->
+      <!-- </collision> -->
+      <xacro:inertial_cuboid mass="${mass*0.98}" xyz="0 0 ${-length/2}"  rpy="0 0 0" x_length="${radius*2}" y_length="${radius*2}" z_length="${length}">
       </xacro:inertial_cuboid>
     </link>
     <link name="${name}_ball_link">
-      <visual>
-      	<origin xyz="0 0 0" rpy="0 0 0"/>
-      	<geometry>
-          <sphere radius="${radius*1.2}"/>
-      	</geometry>
-      	<xacro:orbita3d_grey/>
-      </visual>
-      <collision>
-      	<origin xyz="0 0 0" rpy="0 0 0"/>
-      	<geometry>
-          <sphere radius="${radius*1.2}"/>
-      	</geometry>
-      </collision>
-      <xacro:inertial_sphere mass="${mass*0.5}" diameter="${2*radius*1.2}"/>
+      <!-- <visual> -->
+      <!-- 	<origin xyz="0 0 0" rpy="0 0 0"/> -->
+      <!-- 	<geometry> -->
+      <!--     <sphere radius="${radius*1.2}"/> -->
+      <!-- 	</geometry> -->
+      <!-- 	<xacro:orbita3d_grey/> -->
+      <!-- </visual> -->
+      <!-- <collision> -->
+      <!-- 	<origin xyz="0 0 0" rpy="0 0 0"/> -->
+      <!-- 	<geometry> -->
+      <!--     <sphere radius="${radius*1.2}"/> -->
+      <!-- 	</geometry> -->
+      <!-- </collision> -->
+      <!-- <xacro:inertial_sphere mass="${mass*0.5}" diameter="${2*radius*1.2}"/> -->
     </link>
     <joint name="${name}_ball_joint" type="fixed">
@@ -60,7 +60,48 @@
       <child link="${name}_ball_link"/>
     </joint>
+    <link name="${name}_base_link">
+      <visual>
+	<origin xyz="0 0 0.0672" rpy="0 0 0"/>
+	<geometry>
+          <cylinder radius="0.0278" length="0.0336"/>
+	</geometry>
+	<xacro:orbita3d_grey/>
+      </visual>
+    </link>
+    <joint name="${name}_base_joint" type="fixed">
+      <!-- <origin xyz="0 0 0" rpy="0 0 0"/> -->
+    <xacro:if value="${name == 'r_wrist'}">
+      <origin xyz="${xyz}" rpy="3.141592 0 1.5707963267948966"/>
+    </xacro:if>
+    <xacro:if value="${name == 'l_wrist'}">
+      <origin xyz="${xyz}" rpy="3.141592 0 1.5707963267948966"/>
+    </xacro:if>
+    <xacro:if value="${name == 'neck'}">
+      <origin xyz="${xyz}" rpy="${rpy}"/>
+    </xacro:if>
+      <parent link="${parent}"/>
+      <child link="${name}_base_link"/>
+    </joint>
+    <link name="${name}_out_link">
+    </link>
+    <joint name="${name}_out_joint" type="fixed">
+      <!-- <origin xyz="0 0 0" rpy="0 0 0"/> -->
+    <xacro:if value="${name == 'r_wrist'}">
+      <origin xyz="0 0 0" rpy="3.141592 0 0"/>
+    </xacro:if>
+    <xacro:if value="${name == 'l_wrist'}">
+      <origin xyz="0 0 0" rpy="3.141592 0 0"/>
+    </xacro:if>
+    <xacro:if value="${name == 'neck'}">
+      <origin xyz="0 0 0" rpy="3.141592 0 0"/>
+    </xacro:if>
+      <parent link="${name}_ball_link"/>
+      <child link="${name}_out_link"/>
+    </joint>
     <joint name="${name}_roll" type="revolute">
-      <origin xyz="${xyz}" rpy="${rpy}"/>
-      <parent link="${parent}"/>
+      <!-- <origin xyz="${xyz}" rpy="${rpy}"/> -->
+      <origin xyz="0 0 0" rpy="0 0 0"/>
+      <!-- <parent link="${parent}"/> -->
+      <parent link="${name}_base_link"/>
       <child link="${name}_dummy_link1"/>
       <axis xyz="1 0 0"/>

Commit message: inverse frame for neck

File: orbita3d_description/urdf/orbita3d.urdf.xacro (robot description, xacro)
@@ -94,5 +94,6 @@
     </xacro:if>
     <xacro:if value="${name == 'neck'}">
-      <origin xyz="0 0 0" rpy="3.141592 0 0"/>
+      <!-- <origin xyz="0 0 0" rpy="3.141592 0 0"/> -->
+      <origin xyz="0 0 0" rpy="0 0 0"/>
     </xacro:if>
       <parent link="${name}_ball_link"/>

Commit message: remove cylinder

File: orbita3d_description/urdf/orbita3d.urdf.xacro (robot description, xacro)
@@ -61,11 +61,11 @@
     </joint>
     <link name="${name}_base_link">
-      <visual>
-	<origin xyz="0 0 0.0672" rpy="0 0 0"/>
-	<geometry>
-          <cylinder radius="0.0278" length="0.0336"/>
-	</geometry>
-	<xacro:orbita3d_grey/>
-      </visual>
+      <!-- <visual> -->
+      <!-- 	<origin xyz="0 0 0.0672" rpy="0 0 0"/> -->
+      <!-- 	<geometry> -->
+      <!--     <cylinder radius="0.0278" length="0.0336"/> -->
+      <!-- 	</geometry> -->
+      <!-- 	<xacro:orbita3d_grey/> -->
+      <!-- </visual> -->
     </link>
     <joint name="${name}_base_joint" type="fixed">

Commit message: wip gazebo

File: orbita3d_description/urdf/orbita3d.urdf.xacro (robot description, xacro)
@@ -7,10 +7,11 @@
     <!--
       Orbita3d
-    link                      (joint)
-    ${parent}                  (${name}_roll)
-      ${name}_dummy_link1      (${name}_pitch)
-        ${name}_dummy_link2    (${name}_yaw)
-          ${name}_link         (${name}_ball_joint)
-            ${name}_ball_link
+    link                         (joint)
+    ${parent}                    (${name}_base_joint) fixed
+      ${name}_base_link          (${name}_roll) revolute
+        ${name}_dummy_link1      (${name}_pitch) revolute
+          ${name}_dummy_link2    (${name}_yaw) revolute
+            ${name}_link         (${name}_ball_joint) fixed
+              ${name}_ball_link
     -->
     <link name="${name}_dummy_link1">
@@ -54,4 +55,9 @@
       <!-- </collision> -->
       <!-- <xacro:inertial_sphere mass="${mass*0.5}" diameter="${2*radius*1.2}"/> -->
+      <inertial>
+        <origin xyz="0.0 0.0 0.0" rpy="0.0 0.0 0.0"/>
+        <mass value="0.001"/>
+        <inertia ixx="1.0e-6" ixy="1.0e-8" ixz="1.0e-8" iyy="1.0e-6" iyz="1.0e-8" izz="1.0e-6"/>
+      </inertial>
     </link>
     <joint name="${name}_ball_joint" type="fixed">
@@ -68,4 +74,9 @@
       <!-- 	<xacro:orbita3d_grey/> -->
       <!-- </visual> -->
+      <inertial>
+        <origin xyz="0.0 0.0 0.0" rpy="0.0 0.0 0.0"/>
+        <mass value="0.001"/>
+        <inertia ixx="1.0e-6" ixy="1.0e-8" ixz="1.0e-8" iyy="1.0e-6" iyz="1.0e-8" izz="1.0e-6"/>
+      </inertial>
     </link>
     <joint name="${name}_base_joint" type="fixed">
@@ -84,4 +95,9 @@
     </joint>
     <link name="${name}_out_link">
+      <inertial>
+        <origin xyz="0.0 0.0 0.0" rpy="0.0 0.0 0.0"/>
+        <mass value="0.001"/>
+        <inertia ixx="1.0e-6" ixy="1.0e-8" ixz="1.0e-8" iyy="1.0e-6" iyz="1.0e-8" izz="1.0e-6"/>
+      </inertial>
     </link>
     <joint name="${name}_out_joint" type="fixed">

Commit message: Update angle limits of O3D.

File: orbita3d_description/urdf/orbita3d.urdf.xacro (robot description, xacro)
@@ -123,5 +123,5 @@
       <child link="${name}_dummy_link1"/>
       <axis xyz="1 0 0"/>
-      <limit lower="-0.35" upper="0.35" effort="1000.0" velocity="100.0"/>
+      <limit lower="-0.70" upper="0.70" effort="1000.0" velocity="100.0"/>
       <dynamics damping="${damping}" friction="${friction}"/>
     </joint>
@@ -131,5 +131,5 @@
       <child link="${name}_dummy_link2"/>
       <axis xyz="0 1 0"/>
-      <limit lower="-0.35" upper="0.35" effort="1000.0" velocity="100.0"/>
+      <limit lower="-0.70" upper="0.70" effort="1000.0" velocity="100.0"/>
       <dynamics damping="${damping}" friction="${friction}"/>
     </joint>
